File: DigitalDelay_Multiplex_Jr_1776pedal/multiplex_jr/multiplex_jr.kicad_sch (KiCad schematic)
At the start: 69 parts, among them SW1 SW_SPST, U1 PT2399, U2 TL072, U4 VTL5C, U5 L78L05_TO92, U6 TL072, U7 TL072, U8 TL072

Commit message: back up of all files
Parts:
- removed C1, C16: 22nF, symbol Device:C
- removed C10, C13, C2: 1uF, symbol Device:C_Polarized
- removed C14: 4.7nF, symbol Device:C
- removed C15, C17: 1nF, symbol Device:C
- removed C18: 10nF, symbol Device:C
- removed C19, C22: 47nF, symbol Device:C
- removed C20, C21, C24, C25: 100nF, symbol Device:C
- removed C23: 47uF, symbol Device:C_Polarized
- removed C7: 10uF, symbol Device:C
- removed C8: 10uF, symbol Device:C_Polarized
- removed C9: 47pF, symbol Device:C
- removed D2, D4: LED, symbol Device:LED
- removed R1, R17: 1M, symbol Device:R_US
- removed R10: 1k, symbol Device:R_US
- removed R11, R5, R6, R9: 100k, symbol Device:R_US
- removed R12: 200k, symbol Device:R_US
- removed R13: 22k, symbol Device:R_US
- removed R14: 12k, symbol Device:R_US
- removed R15: 20k, symbol Device:R_US
- removed R18, R19, R20, R26: 10k, symbol Device:R_US
- removed R27: 2.7k, symbol Device:R_US
- removed R7: 47k, symbol Device:R_US
- removed R8: 2.2M, symbol Device:R_US
- removed RV1, RV2: 50k, symbol Device:R_Potentiometer
- removed RV3: 100k, symbol Device:R_Potentiometer
- removed SW1: SW_SPST, symbol Switch:SW_SPST
- removed U1: PT2399, symbol Audio:PT2399
- removed U2, U6, U7, U8: TL072, symbol Amplifier_Operational:TL072
- added C27: 47uF, Capacitor_THT:CP_Radial_D8.0mm_P3.50mm, symbol Device:C_Polarized
- added C28, C29, C33, C36: 100nF, Capacitor_THT:C_Disc_D4.7mm_W2.5mm_P5.00mm, symbol Device:C
- added C31: 4.7nF, Capacitor_THT:C_Disc_D4.7mm_W2.5mm_P5.00mm, symbol Device:C
- added C32, C34: 1nF, Capacitor_THT:C_Disc_D4.7mm_W2.5mm_P5.00mm, symbol Device:C
- added C35, C39, C42, C43: 1uF, Capacitor_THT:CP_Radial_D8.0mm_P3.50mm, symbol Device:C_Polarized
- added C37, C44: 47nF, Capacitor_THT:C_Disc_D4.7mm_W2.5mm_P5.00mm, symbol Device:C
- added C38: 100pF, Capacitor_THT:C_Disc_D4.7mm_W2.5mm_P5.00mm, symbol Device:C
- added C40, C45: 22nF, Capacitor_THT:C_Disc_D4.7mm_W2.5mm_P5.00mm, symbol Device:C
- added C41: 10nF, Capacitor_THT:C_Disc_D4.7mm_W2.5mm_P5.00mm, symbol Device:C
- added C46: 47pF, Capacitor_THT:C_Disc_D4.7mm_W2.5mm_P5.00mm, symbol Device:C
- added D6, D7: LED, LED_THT:LED_D3.0mm, symbol Device:LED
- added J1: Barrel_Jack, Connector_BarrelJack:BarrelJack_Wuerth_6941xx301002, symbol Connector:Barrel_Jack
- added R30: 2.7k, Resistor_THT:R_Axial_DIN0207_L6.3mm_D2.5mm_P10.16mm_Horizontal, symbol Device:R_US
- added R33, R34, R35, R36, R38: 10k, Resistor_THT:R_Axial_DIN0207_L6.3mm_D2.5mm_P10.16mm_Horizontal, symbol Device:R_US
- added R37: 22k, Resistor_THT:R_Axial_DIN0207_L6.3mm_D2.5mm_P10.16mm_Horizontal, symbol Device:R_US
- added R39: 5k, Resistor_THT:R_Axial_DIN0207_L6.3mm_D2.5mm_P10.16mm_Horizontal, symbol Device:R_US
- added R40, R41: 20k, Resistor_THT:R_Axial_DIN0207_L6.3mm_D2.5mm_P10.16mm_Horizontal, symbol Device:R_US
- added R42, R45: 1k, Resistor_THT:R_Axial_DIN0207_L6.3mm_D2.5mm_P10.16mm_Horizontal, symbol Device:R_US
- added R43: 12k, Resistor_THT:R_Axial_DIN0207_L6.3mm_D2.5mm_P10.16mm_Horizontal, symbol Device:R_US
- added R44: 2k, Resistor_THT:R_Axial_DIN0207_L6.3mm_D2.5mm_P10.16mm_Horizontal, symbol Device:R_US
- added R46, R47: 1M, Resistor_THT:R_Axial_DIN0207_L6.3mm_D2.5mm_P10.16mm_Horizontal, symbol Device:R_US
- added R48: 100k, Resistor_THT:R_Axial_DIN0207_L6.3mm_D2.5mm_P10.16mm_Horizontal, symbol Device:R_US
- added R49: 200k, Resistor_THT:R_Axial_DIN0207_L6.3mm_D2.5mm_P10.16mm_Horizontal, symbol Device:R_US
- added RV6, RV7, RV8: 50k, Potentiometer_THT:Potentiometer_Piher_T-16H_Single_Horizontal, symbol Device:R_Potentiometer
- added SW3: SW_SPST, symbol Switch:SW_SPST
- added U3: ~, Package_DIP:DIP-8_W7.62mm, symbol New_Library:TL072P
- added U8: ~, Package_TO_SOT_THT:TO-92_Inline, symbol New_Library:TL072P
- added U9: PT2399, Package_DIP:DIP-16_W7.62mm, symbol Audio:PT2399
- C11: value 100pF -> 10uF; footprint (none) -> Capacitor_THT:C_Disc_D4.7mm_W2.5mm_P5.00mm
- C12: value 1uF -> 10uF; footprint (none) -> Capacitor_THT:CP_Radial_D8.0mm_P3.50mm
- C3, C4, C5, C6: footprint (none) -> Capacitor_THT:CP_Radial_D8.0mm_P3.50mm
- R16, R2, R28, R3, R4: footprint (none) -> Resistor_THT:R_Axial_DIN0207_L6.3mm_D2.5mm_P10.16mm_Horizontal
- R21: value 5k -> 100k; footprint (none) -> Resistor_THT:R_Axial_DIN0207_L6.3mm_D2.5mm_P10.16mm_Horizontal
- R22: value 10k -> 100k; footprint (none) -> Resistor_THT:R_Axial_DIN0207_L6.3mm_D2.5mm_P10.16mm_Horizontal
- R23: value 20k -> 47k; footprint (none) -> Resistor_THT:R_Axial_DIN0207_L6.3mm_D2.5mm_P10.16mm_Horizontal
- R24: value 1k -> 100k; footprint (none) -> Resistor_THT:R_Axial_DIN0207_L6.3mm_D2.5mm_P10.16mm_Horizontal
- R25: value 2k -> 2.2M; footprint (none) -> Resistor_THT:R_Axial_DIN0207_L6.3mm_D2.5mm_P10.16mm_Horizontal
- RV4: value 50k -> 100k; footprint (none) -> Potentiometer_THT:Potentiometer_Piher_T-16H_Single_Horizontal
- RV5: footprint (none) -> Potentiometer_THT:Potentiometer_Piher_T-16H_Single_Horizontal
Connections:
- net +9V: now also J1.1
- net GND: now also C12.2, R22.2, C27.2, C28.1, C29.2, C31.1, C37.2, C41.1, C44.1, D7.1 (K), J1.2, R46.1, R47.2, RV6.1, RV7.1, RV8.1, U3.4 (Vcc-), U8.4 (Vcc-), U9.3 (AGND), U9.4 (DGND); no longer RV4.1
- net IN: now also C45.1, R47.1
- net MOD IN: now also R30.2, RV6.2, RV6.3; no longer RV4.2, RV4.3
- net OUT: now also R45.2, R46.2; no longer R16.2
- net Va: now also R21.1, U3.8 (Vcc+), U8.8 (Vcc+)
- net Vb: now also U3.3 (1IN+), U3.5 (2IN+)
- net Vc: now also U9.1 (VCC)
- net at C11.2: now also R24.1, U8.2 (1IN-)
- net at C11.1: now also R23.2, RV4.3, U8.1 (1OUT)
- net at R21.2: now also R22.1, R23.1, U8.3 (1IN+)
- net at C12.1: now also R24.2, R25.1, RV4.1, RV4.2
- net at R16.1: now also U8.6 (2IN-), U8.7 (2OUT)
- net at R25.2: now also U8.5 (2IN+)
- new net: C45.2, R48.1
- new net: C39.2, RV7.2
- new net: C42.2, R44.2, RV7.3
- new net: C33.1, U9.10 (OP1-IN)
- new net: C33.2, U9.9 (OP1-OUT)
- new net: C46.1, R48.2, R49.1, U3.2 (1IN-)
- new net: C39.1, R40.2
- new net: C44.2, R44.1, RV8.2
- new net: C29.1, U9.8 (CC0)
- new net: C37.1, R36.2, R38.1, R41.1
- new net: D7.2 (A), SW3.2 (B)
- new net: C32.1, R35.2, U9.15 (LPF1-OUT)
- new net: C32.2, R33.2, U9.16 (LPF1-IN)
- new net: C38.1, R37.2, R40.1, R43.1, U3.6 (2IN-)
- new net: C35.1, R37.1
- new net: C34.1, R36.1, U9.13 (LPF2-IN)
- new net: C34.2, R41.2, R42.1, U9.14 (LPF2-OUT)
- new net: C46.2, R49.2, U3.1 (1OUT)
- new net: D6.1 (K), SW3.1 (A)
- new net: D6.2 (A), R16.2
- new net: C27.1, U9.2 (REF)
- new net: C31.2, R33.1, R34.2, R35.1, R39.1
- new net: C35.2, R34.1
- new net: C36.1, R38.2, U9.12 (OP2-OUT)
- new net: C36.2, U9.11 (OP2-IN)
- new net: C41.2, C42.1, R42.2
- new net: R30.1, U9.6 (VCO)
- new net: C28.2, U9.7 (CC1)
- new net: C38.2, C43.1, R43.2, U3.7 (2OUT)
- new net: C40.1, RV8.3
- new net: C43.2, R45.1
- new net: C40.2, R39.2
Other:
- note added: "1.3V"
- note added: "DEPTH"
- note added: "Feedback"
- note added: "MIX"
- note added: "Power Supply and Voltage Regulation"
- note added: "SPEED"
- note added: "Signal Processing and Modulation"
- moved on the sheet: R28, RV5, U4
